File: PWR.kicad_sch (KiCad schematic)
At the start: 51 parts, among them U1 TI_TLV743P, U2 Ti_TPS566238

Commit message: Version 1.1
Parts:
- removed C11, C13, C22: 47u, Capacitor_SMD:CP_Elec_6.3x5.8, symbol Device:C_Polarized_Small
- removed C15, C16, C5, C6: 22u, Capacitor_SMD:CP_Elec_6.3x5.4_Nichicon, symbol Device:C_Polarized_Small
- removed C18, C31, C7, C8: 100n, Capacitor_SMD:C_0402_1005Metric, symbol Device:C_Small
- removed C32, C33, C34: 100n, Capacitor_SMD:C_1206_3216Metric, symbol Device:C_Small
- removed H2, H4, H5, H6, H7, H8: ~, MountingHole:MountingHole_4.3mm_M4_Pad_TopBottom, symbol Mechanical:MountingHole_Pad
- removed L1: 1.5u, Inductor_SMD:L_Coilcraft_XAL1010-XXX, symbol Device:L_Small
- removed U2: Ti_TPS566238, Library:Ti_RQF0009A, symbol Library:Ti_TPS566238
- added C1, C11, C2, C20, C21: 22u, Capacitor_SMD:C_0805_2012Metric, symbol Device:C_Small
- added C13, C14, C4, C5: 22u, Capacitor_SMD:C_0603_1608Metric, symbol Device:C_Small
- added C24: 100n, Capacitor_SMD:C_0402_1005Metric, symbol Device:C_Small
- added J6: PWR_IN, Library:XKB_X9357WR-2x02-N2SN, symbol Connector_Generic:Conn_02x02_Top_Bottom
- added U2, U3: TPS82130, Package_LGA:Texas_SIL0008D_MicroSiP-8-1EP_2.8x3mm_P0.65mm_EP1.1x1.9mm_ThermalVias, symbol Regulator_Switching:TPS82130
- C12: value 100n -> 22u; footprint Capacitor_SMD:C_0402_1005Metric -> Capacitor_SMD:C_0805_2012Metric; LCSC C105883 -> C602037; PN CC0402KRX7R8BB104 -> CL21A226MAYNNNE; Vendor YAGEO -> Samsung
- C25: value 1u -> 100n; footprint Capacitor_SMD:C_0402_1005Metric -> Capacitor_SMD:C_1206_3216Metric; LCSC C52923 -> C23631; PN CL05A105KA5NQNC -> CC1206KKX7RDBB102; Vendor Samsung -> YAGEO
- C26: value 10n -> 100n; footprint Capacitor_SMD:C_0402_1005Metric -> Capacitor_SMD:C_1206_3216Metric; LCSC C60133 -> C23631; PN CC0402KRX7R9BB103 -> CC1206KKX7RDBB102
- C27: value 100n -> 22u; footprint Capacitor_SMD:C_0402_1005Metric -> Capacitor_SMD:C_0603_1608Metric; LCSC C60474 -> C159801; PN CC0402KRX7R7BB104 -> CL10A226MQ8NRNE; Vendor YAGEO -> Samsung
- C28: value 100n -> 22u; footprint Capacitor_SMD:C_1206_3216Metric -> Capacitor_SMD:C_0603_1608Metric; LCSC C23631 -> C159801; PN CC1206KKX7RDBB102 -> CL10A226MQ8NRNE; Vendor YAGEO -> Samsung
- C29: value 33p -> 100n; LCSC C107005 -> C60474; PN CC0402JRNPO9BN330 -> CC0402KRX7R7BB104
- C30: value 22u -> 100n; footprint Capacitor_SMD:C_0603_1608Metric -> Capacitor_SMD:C_0402_1005Metric; LCSC C159801 -> C60474; PN CL10A226MQ8NRNE -> CC0402KRX7R7BB104; Vendor Samsung -> YAGEO
- R11: value 220k -> 523k; LCSC C138030 -> C227128; PN RC0402FR-07220KL -> AC0402FR-07523KL
- R12, R14: value 1M -> 100k; footprint Resistor_SMD:R_0603_1608Metric -> Resistor_SMD:R_0402_1005Metric; LCSC C144621 -> C60491; PN AC0603JR-071ML -> RC0402FR-07100KL
- R13: value 1M -> 523k; footprint Resistor_SMD:R_0603_1608Metric -> Resistor_SMD:R_0402_1005Metric; LCSC C144621 -> C227128; PN AC0603JR-071ML -> AC0402FR-07523KL
- R9: value 30k -> 1M; footprint Resistor_SMD:R_0402_1005Metric -> Resistor_SMD:R_0603_1608Metric; LCSC C138008 -> C144621; PN RC0402FR-0730KL -> AC0603JR-071ML
- renumbered C1 to C10, C19 to C15, C20 to C16, C14 to C18, C21 to C19, C24 to C22, C9 to C6, C10 to C7, C2 to C8, C4 to C9, H3 to H2
Connections:
- net +12V: now also C17.2, C8.2, C1.2, C11.2, C2.1, C20.1, C21.1, C24.1, J6.3 (Pin_3), J6.4 (Pin_4), U2.1 (EN), U2.2 (VIN), U3.1 (EN), U3.2 (VIN); no longer C17.1, C8.1
- net +5V: now also C27.1, C28.1, C29.1, R13.1, C13.2, C14.1, C4.2, C5.1, U2.4 (VOUT), U2.5 (VOUT), U3.4 (VOUT), U3.5 (VOUT); no longer C29.2
- net GND: now also C17.1, C25.2, C27.2, C29.2, C8.1, C1.1, C11.1, C13.1, C14.2, C2.2, C20.2, C21.2, C24.2, C4.1, C5.2, J6.1 (Pin_1), J6.2 (Pin_2), U2.3 (GND), U2.9 (GND), U3.3 (GND), U3.9 (GND); no longer C17.2, C25.1, C8.2, R13.2
- net SH: now reaches C26.1
- net SH: now also C25.1, H1.1, H2.1, R10.1, R9.1
- removed net E1: H1.1, R13.1
- net E2: no longer names the net of R12.1
- net E2: now also R11.2, U2.6 (FB)
- net E3: no longer names the net of R14.1
- net E3: now also R13.2, U3.6 (FB); no longer H2.1
- removed net E4: C28.1, R10.1
- no-connect marks 1 -> 4
Other:
- note added: "12V IN"
- note added: "Change log: - Use TPS82130 for conversion for lower price & BOM count - 12V: Use 47uF capacitor for input only - Power input switch to ATX 4 pin"
- note added: "Chassis - GND M4"
- note added: "INPUT"
- note removed: "12V IN - M4"
- note removed: "Chassis - GND"
- note removed: "DRC"
- note removed: "Mounting Hole - M4"
- title: SAS_Backplane - PWR -> Backplane - PWR
- moved on the sheet: C10, C17, C18, C8, C9, H1, H2
